File: hardware/lamp-sconce/kicad/led_group.sch (KiCad schematic (older format))
At the start: 0 parts

Commit message: Adding more work for the sconce lamp.  Schematic is pretty much complete.
Signed-off-by: Daniel P Williams <dwilliams@port8080.net>
Parts:
- added D47, D48, D49, D50, D51, D52, D53, D54, D55, D56: LED, symbol LED
- added Q13, Q14, Q15: MOSFET_N, symbol MOSFET_N
- added R48, R50, R52: 1Kohm, symbol R
- added R49, R62, R63: 75 ohm, symbol R
- added R51, R53: 10 ohm, symbol R
Connections:
- new net: D47.2 (K), D48.1 (A)
- new net: D48.2 (K), D49.1 (A)
- new net: D51.2 (K), D52.1 (A)
- new net: D54.2 (K), D55.1 (A)
- new net: D55.2 (K), D56.1 (A)
- new net: D52.2 (K), D53.1 (A)
- new net: D49.2 (K), D50.1 (A)
- new net: D50.2 (K), R49.1, R62.1, R63.1
- new net: D53.2 (K), R51.1
- new net: D56.2 (K), R53.1
- new net: Q13.D, R49.2, R62.2, R63.2
- new net: Q14.D, R51.2
- new net: Q15.D, R53.2
- new net: Q15.G, R52.2
- new net: Q14.G, R50.2
- new net: Q13.G, R48.2
- new net LED_+12V: D47.1 (A), D51.1 (A), D54.1 (A)
- new net LED_BLU: R50.1
- new net LED_GND: Q13.S, Q14.S, Q15.S
- new net LED_GRN: R52.1
- new net LED_RED: R48.1
Other:
- note added: "BLU\n140mA\n3.6V"
- note added: "GRN\n140mA\n3.6V"
- note added: "RED\n140mA\n2.1V"
