File: hardware/lamp-sconce/kicad/power_supply.sch (KiCad schematic (older format))
At the start: 0 parts

Commit message: Adding more work for the sconce lamp.  Schematic is pretty much complete.
Signed-off-by: Daniel P Williams <dwilliams@port8080.net>
Parts:
- added C1: 220uF 100V, symbol CP1
- added C2: 0.22uF 100V, symbol C
- added C3, C4: 0.01uF 100V, symbol C
- added C5, C6: 220uF 25V, symbol CP1
- added D41, D42: 60V 3A, symbol DIODESCH
- added L1, L2: 180uH, symbol INDUCTOR
- added R30: 80Kohm, symbol R
- added R31: 50Kohm, symbol R
- added R32: 6.25Kohm, symbol R
- added R33, R35: 2Kohm, symbol R
- added R34: 28Kohm, symbol R
- added SW1: SWITCH_INV, symbol SWITCH_INV
- added U2, U3: A8498, symbol A8498
Connections:
- new net: C3.1, U2.1 (BOOT)
- new net: SW1.2, U2.2 (ENB), U3.2 (ENB)
- new net: R30.1, U2.3 (TSET)
- new net: R32.2, R33.1, U2.5 (FB)
- new net: C3.2, D41.2 (K), L1.1, U2.7 (LX)
- new net: R34.2, R35.1, U3.5 (FB)
- new net: C4.2, D42.2 (K), L2.1, U3.7 (LX)
- new net: C4.1, U3.1 (BOOT)
- new net: R31.1, U3.3 (TSET)
- new net GND: C1.2, C2.2, C5.2, C6.2, D41.1 (A), D42.1 (A), R30.2, R31.2, R33.2, R35.2, SW1.1, U2.4 (GND), U3.4 (GND)
- new net PSU_+12V: C6.1, L2.2, R34.1, U3.6 (VBIAS)
- new net PSU_+3V3: C5.1, L1.2, R32.1
- new net PSU_VIN: C1.1, C2.1, U2.8 (VIN), U3.8 (VIN)
- no-connect marks 0 -> 1
